Commit message: visual upright fix

File: src/eca_a9_description/urdf/eca_a9_visual.urdf.xacro (robot description, xacro)
@@ -7,5 +7,5 @@
   <link name="base_link">
     <visual>
-      <origin xyz="0 0 0" rpy="0 0 0"/>
+      <origin xyz="0 0 0" rpy="3.14159 0 0"/>
       <geometry>
         <mesh filename="${visual_mesh}" scale="1 1 1"/>

Commit message: debugged camera_info + initial tf2 listener

File: src/eca_a9_description/urdf/eca_a9_visual.urdf.xacro (robot description, xacro)
@@ -24,3 +24,21 @@
     </inertial>
   </link>
+  <!-- Forward-Looking Sonar (FLS) frame -->
+  <joint name="base_to_sonar" type="fixed">
+    <parent link="base_link"/>
+    <child link="sonar"/>
+    <!-- Mount at front of vehicle, angled down 90 degrees for testing -->
+    <origin xyz="0.5 0 0" rpy="0 -1.5708 0"/>
+  </joint>
+  <link name="sonar">
+    <visual>
+      <origin xyz="0 0 0" rpy="0 0 0"/>
+      <geometry>
+        <box size="0.05 0.05 0.05"/>
+      </geometry>
+      <material name="sonar_blue">
+        <color rgba="0.0 0.5 1.0 0.8"/>
+      </material>
+    </visual>
+  </link>
 </robot>

Commit message: meshes, interactive marker, and depth fix

File: src/eca_a9_description/urdf/eca_a9_visual.urdf.xacro (robot description, xacro)
@@ -28,6 +28,6 @@
     <parent link="base_link"/>
     <child link="sonar"/>
-    <!-- Mount at front of vehicle, angled down 90 degrees for testing -->
-    <origin xyz="0.5 0 0" rpy="0 -1.5708 0"/>
+    <!-- Mount at base_link, angled down 90 degrees for testing -->
+    <origin xyz="0 0 0" rpy="0 -1.5708 0"/>
   </joint>
   <link name="sonar">
@@ -42,3 +42,11 @@
     </visual>
   </link>
+  <!-- Sonar optical frame (for raycasting coordinate system) -->
+  <!-- Converts to optical convention: +X right, +Y down, +Z forward -->
+  <joint name="sonar_to_optical" type="fixed">
+    <parent link="sonar"/>
+    <child link="sonar_optical"/>
+    <origin xyz="0 0 0" rpy="-1.5708 0 -1.5708"/>
+  </joint>
+  <link name="sonar_optical"/>
 </robot>

Commit message: working run of behaviorized nbv

File: src/eca_a9_description/urdf/eca_a9_visual.urdf.xacro (robot description, xacro)
@@ -28,6 +28,6 @@
     <parent link="base_link"/>
     <child link="sonar"/>
-    <!-- Mount at base_link, angled down 90 degrees for testing -->
-    <origin xyz="0 0 0" rpy="0 -1.5708 0"/>
+    <!-- Mount at bow (0.7m forward), angled down 45 degrees -->
+    <origin xyz="0.7 0 0" rpy="0 -0.7854 0"/>
   </joint>
   <link name="sonar">

Commit message: testing out ARL params

File: src/eca_a9_description/urdf/eca_a9_visual.urdf.xacro (robot description, xacro)
@@ -1,4 +1,9 @@
 <?xml version="1.0"?>
 <robot name="eca_a9_visual" xmlns:xacro="http://ros.org/wiki/xacro">
+  <!-- FLS down-tilt from horizontal, in degrees. Single source of truth for the
+       physical mount angle. Keep this in sync with the helix sampler's
+       mount_angle_deg port (nbv_on_target.xml) and the search server's
+       mount_angle, since those re-aim viewpoints assuming this tilt. -->
+  <xacro:property name="fls_mount_angle_deg" value="20"/>
   <!-- Mesh properties -->
   <xacro:property name="visual_mesh"    value="package://eca_a9_description/mesh/eca_a9.dae"/>
@@ -28,6 +33,7 @@
     <parent link="base_link"/>
     <child link="sonar"/>
-    <!-- Mount at bow (0.7m forward), angled down 45 degrees -->
-    <origin xyz="0.7 0 0" rpy="0 -0.7854 0"/>
+    <!-- Mount at bow (0.7m forward), angled down by fls_mount_angle_deg.
+         Negative pitch tilts the sonar's forward (+X) axis downward. -->
+    <origin xyz="0.7 0 0" rpy="0 ${radians(-fls_mount_angle_deg)} 0"/>
   </joint>
   <link name="sonar">
